File: pcb/tiny-vga.kicad_pcb (KiCad board)
At the start: 2 copper layers, 40 x 33 mm, 32 parts, among them J1 PMOD, J2 VGA, U1 74LVC245APW,118

Commit message: Add "Designed for Tiny Tapeout" logo
Parts:
- removed the REF** at (145.4, 84.2)
- added REF**: KiCad-Logo2_5mm_SilkScreen, Symbol:KiCad-Logo2_5mm_SilkScreen, B.Cu at (154.1, 71.8)
- added REF**: PMOD_LOGO, tiny-vga:TT_PMOD_Logo_10mm, B.Cu at (141.6, 84.6)
- moved REF** 16.0 mm to (153.8, 84.7)
Other:
- board text added: "© Leo Moser 2024, CC BY-SA 4.0"
